Commit message: reverted upstream changes

File: models/rotors_description/urdf/component_snippets.xacro (robot description, xacro)
@@ -128,5 +128,5 @@
   </xacro:macro>
   <!-- Macro to add the mavlink interface. -->
-  <xacro:macro name="mavlink_interface_macro" params="namespace imu_sub_topic gps_sub_topic mavlink_addr mavlink_udp_port serial_enabled serial_device baudrate qgc_addr qgc_udp_port hil_mode hil_state_level vehicle_is_tailsitter send_vision_estimation send_odometry enable_lockstep use_tcp">
+  <xacro:macro name="mavlink_interface_macro" params="namespace imu_sub_topic gps_sub_topic mavlink_addr mavlink_udp_port serial_enabled serial_device baudrate qgc_addr qgc_udp_port hil_mode hil_state_level vehicle_is_tailsitter send_odometry">
     <gazebo>
       <plugin name="mavlink_interface" filename="libgazebo_mavlink_interface.so">
@@ -144,8 +144,5 @@
         <hil_state_level>$(arg hil_state_level)</hil_state_level>
         <vehicle_is_tailsitter>$(arg vehicle_is_tailsitter)</vehicle_is_tailsitter>
-        <send_vision_estimation>$(arg send_vision_estimation)</send_vision_estimation>
         <send_odometry>$(arg send_odometry)</send_odometry>
-        <enable_lockstep>$(arg enable_lockstep)</enable_lockstep>
-        <use_tcp>$(arg use_tcp)</use_tcp>
         <motorSpeedCommandPubTopic>/gazebo/command/motor_speed</motorSpeedCommandPubTopic>
         <control_channels>

File: models/rotors_description/urdf/iris_base.xacro (robot description, xacro)
@@ -14,8 +14,5 @@
   <xacro:arg name='hil_mode' default='false' />
   <xacro:arg name='hil_state_level' default='false' />
-  <xacro:arg name='send_vision_estimation' default='false' />
   <xacro:arg name='send_odometry' default='false' />
-  <xacro:arg name='enable_lockstep' default='true' />
-  <xacro:arg name='use_tcp' default='true' />
   <xacro:arg name='vehicle_is_tailsitter' default='false' />
   <xacro:arg name='visual_material' default='DarkGrey' />
@@ -64,8 +61,5 @@
     hil_state_level="$(arg hil_state_level)"
     vehicle_is_tailsitter="$(arg vehicle_is_tailsitter)"
-    send_vision_estimation="$(arg send_vision_estimation)"
     send_odometry="$(arg send_odometry)"
-    enable_lockstep="$(arg enable_lockstep)"
-    use_tcp="$(arg use_tcp)"
     >
   </xacro:mavlink_interface_macro>
